File: board/board.sch (KiCad schematic (older format))
At the start: 21 parts, among them J1 Conn_01x02, J2 Conn_01x02, J3 Conn_01x02, J4 Conn_02x02_Top_Bottom, J5 Conn_02x05_Top_Bottom

Commit message: pcb layout completed
Parts:
- J4: symbol Connector_Generic:Conn_02x02_Top_Bottom -> Connector_Generic:Conn_02x02_Odd_Even
- J5: symbol Connector_Generic:Conn_02x05_Top_Bottom -> Connector_Generic:Conn_02x05_Odd_Even
Connections:
- net ~V_SHDN: now also J4.3 (Pin_3); no longer J4.2 (Pin_2)
- net at D1.2 (A), J5.1 (Pin_1), J5.3 (Pin_3)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: now also J5.7 (Pin_7), J5.9 (Pin_9); no longer J5.2 (Pin_2), J5.4 (Pin_4)
- net at D1.1 (K), J4.4 (Pin_4), R1.2: now also J4.2 (Pin_2); no longer J4.3 (Pin_3)
- net at C4.2: now also J5.6 (Pin_6); no longer J5.8 (Pin_8)
- net at C3.2: now also J5.4 (Pin_4); no longer J5.7 (Pin_7)
- net at C5.2: now also J5.8 (Pin_8); no longer J5.9 (Pin_9)
- net at C2.2: now also J5.2 (Pin_2); no longer J5.6 (Pin_6)
Changed lines of the file:
@@
 $EndComp
 $Comp
-L Connector_Generic:Conn_02x05_Top_Bottom J5
+L Connector_Generic:Conn_02x05_Odd_Even J5
 U 1 1 611C6950
 P 4450 6400
@@
 	7200 4050 7200 6400
 $Comp
-L Connector_Generic:Conn_02x02_Top_Bottom J4
+L Connector_Generic:Conn_02x02_Odd_Even J4
 U 1 1 611F47B2
 P 3100 4600

Commit message: minor changes i guess
Parts:
- D1: value 1N4148WT -> 1N4148
- D2: value MBR0520LT3G -> MBR0520; Manufacturer/Part Number MBR0520LT3G -> MBR0520L-TP; Supplier Stock Code 863-MBR0520LT3G -> 833-MBR0520L-TP
Changed lines of the file:
@@
 P 6600 3850
 F 0 "D2" V 6646 3770 50  0000 R CNN
-F 1 "MBR0520LT3G" V 6555 3770 50  0000 R CNN
+F 1 "MBR0520" V 6555 3770 50  0000 R CNN
 F 2 "Diode_SMD:D_SOD-123" H 6600 3850 50  0001 C CNN
 F 3 "https://www.mouser.it/datasheet/2/308/1/MBR0520LT1_D-2315148.pdf" H 6600 3850 50  0001 C CNN
-F 4 "MBR0520LT3G" H 6600 3850 50  0001 C CNN "Manufacturer/Part Number"
-F 5 "863-MBR0520LT3G" H 6600 3850 50  0001 C CNN "Supplier Stock Code"
+F 4 "MBR0520L-TP" H 6600 3850 50  0001 C CNN "Manufacturer/Part Number"
+F 5 "833-MBR0520L-TP" H 6600 3850 50  0001 C CNN "Supplier Stock Code"
 	1    6600 3850
 	0    -1   -1   0
@@
 P 3950 5050
 F 0 "D1" H 3950 5267 50  0000 C CNN
-F 1 "1N4148WT" H 3950 5176 50  0000 C CNN
+F 1 "1N4148" H 3950 5176 50  0000 C CNN
 F 2 "Diode_SMD:D_SOD-523" H 3950 4875 50  0001 C CNN
 F 3 "https://assets.nexperia.com/documents/data-sheet/1N4148_1N4448.pdf" H 3950 5050 50  0001 C CNN
